Commit message: update ik

File: resources/robots/wow_little/urdf/up_body_wo_dummy.urdf (robot description, URDF)
Before this commit: robot up_body, 17 links, 16 joints
Links:
- link base: geometry collision mesh filename=../meshes/base.STL; visual mesh filename=../meshes/base.STL
- link left_1_link: geometry collision mesh filename=../meshes/left_1_link.STL; visual mesh filename=../meshes/left_1_link.STL
- link left_2_link: geometry collision mesh filename=../meshes/left_2_link.STL; visual mesh filename=../meshes/left_2_link.STL
- link left_3_link: geometry collision mesh filename=../meshes/left_3_link.STL; visual mesh filename=../meshes/left_3_link.STL
- link left_4_link: geometry collision mesh filename=../meshes/left_4_link.STL; visual mesh filename=../meshes/left_4_link.STL
- link left_5_link: geometry collision mesh filename=../meshes/left_5_link.STL; visual mesh filename=../meshes/left_5_link.STL
- link left_6_link: geometry collision mesh filename=../meshes/left_6_link.STL; visual mesh filename=../meshes/left_6_link.STL
- link left_7_link: geometry collision mesh filename=../meshes/left_7_link.STL; visual mesh filename=../meshes/left_7_link.STL
- link left_8_link: geometry collision mesh filename=../meshes/left_8_link.STL; visual mesh filename=../meshes/left_8_link.STL
- link right_1_link: geometry collision mesh filename=../meshes/right_1_link.STL; visual mesh filename=../meshes/right_1_link.STL
- link right_2_link: geometry collision mesh filename=../meshes/right_2_link.STL; visual mesh filename=../meshes/right_2_link.STL
- link right_3_link: geometry collision mesh filename=../meshes/right_3_link.STL; visual mesh filename=../meshes/right_3_link.STL
- link right_4_link: geometry collision mesh filename=../meshes/right_4_link.STL; visual mesh filename=../meshes/right_4_link.STL
- link right_5_link: geometry collision mesh filename=../meshes/right_5_link.STL; visual mesh filename=../meshes/right_5_link.STL
- link right_6_link: geometry collision mesh filename=../meshes/right_6_link.STL; visual mesh filename=../meshes/right_6_link.STL
- link right_7_link: geometry collision mesh filename=../meshes/right_7_link.STL; visual mesh filename=../meshes/right_7_link.STL
- link right_8_link: geometry collision mesh filename=../meshes/right_8_link.STL; visual mesh filename=../meshes/right_8_link.STL
Joints:
- joint left_1_joint: limit lower=-1.22 upper=2.2 effort=0 velocity=3 -> lower=-1.22 upper=2.2 effort=30 velocity=3
- joint left_2_joint: limit lower=-1.5 upper=0.2 effort=0 velocity=3 -> lower=-1.5 upper=0.2 effort=30 velocity=3
- joint left_3_joint: limit lower=-2.5 upper=2.5 effort=0 velocity=3 -> lower=-2.5 upper=2.5 effort=30 velocity=3
- joint left_4_joint: limit lower=-1.75 upper=1.75 effort=0 velocity=3 -> lower=-1.75 upper=1.75 effort=30 velocity=3
- joint left_5_joint: limit lower=-3 upper=3 effort=0 velocity=3 -> lower=-3 upper=3 effort=30 velocity=3
- joint left_6_joint: limit lower=-1.75 upper=1.75 effort=0 velocity=3 -> lower=-1.75 upper=1.75 effort=30 velocity=3
- joint left_7_joint: limit lower=-1.75 upper=1.75 effort=0 velocity=3 -> lower=-1.75 upper=1.75 effort=30 velocity=3
- joint left_8_joint: limit lower=-3 upper=3 effort=0 velocity=3 -> lower=-3 upper=3 effort=30 velocity=3
- joint right_1_joint: limit lower=-2.2 upper=1.22 effort=0 velocity=3 -> lower=-2.2 upper=1.22 effort=30 velocity=3
- joint right_2_joint: limit lower=-1.5 upper=0.2 effort=0 velocity=3 -> lower=-1.5 upper=0.2 effort=30 velocity=3
- joint right_3_joint: limit lower=-2.5 upper=2.5 effort=0 velocity=3 -> lower=-2.5 upper=2.5 effort=30 velocity=3
- joint right_4_joint: limit lower=-1.75 upper=1.75 effort=0 velocity=3 -> lower=-1.75 upper=1.75 effort=30 velocity=3
- joint right_5_joint: limit lower=-3 upper=3 effort=0 velocity=3 -> lower=-3 upper=3 effort=30 velocity=3
- joint right_6_joint: limit lower=-1.75 upper=1.75 effort=0 velocity=3 -> lower=-1.75 upper=1.75 effort=30 velocity=3
- joint right_7_joint: limit lower=-1.75 upper=1.75 effort=0 velocity=3 -> lower=-1.75 upper=1.75 effort=30 velocity=3
- joint right_8_joint: limit lower=-3 upper=3 effort=0 velocity=3 -> lower=-3 upper=3 effort=30 velocity=3
